File: Mixer_KiCAD/Mixer/Mixer.kicad_sch (KiCad schematic)
At the start: 63 parts, among them IC1 HMC220BMS8GETR, IC2 LMX2572RHAT, IC3 HMC220BMS8GETR, IC4 TPS74601PQWDRBRQ1, IC5 MCP2210-I_MQ, J1 CONSMA020.062-G, J2 CONSMA020.062-G, J3 CONSMA020.062-G, J4 CONSMA020.062-G, J5 USB4940-00-A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

Commit message: updated BOM
Parts:
- C1, C11, C12, C19: Distributor Link (none) -> https://www.mouser.com/ProductDetail/Murata-Electronics/GRM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; MPN (none) -> GRM155R70J104KA01D
- C10, C24, C31, C8, C9: Distributor Link (none) -> https://www.mouser.com/ProductDetail/Murata-Electronics/GRT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; MPN (none) -> GRT155C80J105KE01D
- C13, C16, C2, C3, C4, C5, C6, C7: Distributor Link (none) -> https://www.mouser.com/ProductDetail/Murata-Electronics/GCM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; MPN (none) -> GCM1555C1H200JA16D
- C14: Distributor Link (none) -> https://www.mouser.com/ProductDetail/KYOCERA-AVX/04026C681K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; MPN (none) -> 04026C681KAT2A
- C15: Distributor Link (none) -> https://www.mouser.com/ProductDetail/Murata-Electronics/GRM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; MPN (none) -> GRM1555C1H152GA01D
- C17: Distributor Link (none) -> https://www.mouser.com/ProductDetail/Murata-Electronics/GRM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; MPN (none) -> GRM155R61A124ME19D
- C18, C21, C23, C30, C33: Distributor Link (none) -> https://www.mouser.com/ProductDetail/Murata-Electronics/GRM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; MPN (none) -> GRM188R60J106ME47D
- C20, C29: Distributor Link (none) -> https://www.mouser.com/ProductDetail/Murata-Electronics/GRM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; MPN (none) -> GRM155R61H474ME11D
- C22, C32: Distributor Link (none) -> https://www.mouser.com/ProductDetail/Murata-Electronics/GRM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; MPN (none) -> GRM155R71E103JA01J
- C25, C26: Distributor Link (none) -> https://www.mouser.com/ProductDetail/Murata-Electronics/GRM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; MPN (none) -> GRM1557U1A302JA01D
- C27, C28: Distributor Link (none) -> https://www.mouser.com/ProductDetail/Murata-Electronics/GCM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; MPN (none) -> GCM1555C1H4R0BA16J
- C34, C35: Distributor Link (none) -> https://www.mouser.com/ProductDetail/Murata-Electronics/GCM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; MPN (none) -> GCM1555C1H100JA16J
- IC2: MPN LMX2572RHAR -> LMX2572RHAT
- R1, R2: Distributor Link (none) -> https://www.mouser.com/ProductDetail/Vishay/TNPW060350R0DEE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; MPN (none) -> TNPW060350R0DEEA
- R3: Distributor Link (none) -> https://www.mouser.com/ProductDetail/Vishay/RCA0603330RFKEA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; MPN (none) -> RCA0603330RFKEASR
- R4: Distributor Link (none) -> https://www.mouser.com/ProductDetail/Vishay-Beyschlag/MCT06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; MPN (none) -> MCT0603MC1200FP500
- R5, R6: Distributor Link (none) -> https://www.mouser.com/ProductDetail/Vishay/CRCW06035K10FKE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; MPN (none) -> CRCW06035K10FKEBC
- R7: Distributor Link (none) -> https://www.mouser.com/ProductDetail/Vishay/CRCW06031M00FKE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; MPN (none) -> CRCW06031M00FKEAC
- R8: Distributor Link (none) -> https://www.mouser.com/ProductDetail/Vishay/CRCW0603140RFKE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; MPN (none) -> CRCW0603140RFKEAC
- R9: Distributor Link (none) -> https://www.mouser.com/ProductDetail/Vishay/CRCW0603200KFKE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; MPN (none) -> CRCW0603200KFKEBC
